File: heart_necklace.sch (EAGLE design)
At the start: 23 parts, among them SW1 300mA/4V

Commit message: Renamed files to heart_necklace.  Added gitignore.  Did most of routing
Connections:
- net LED1: now also LED9.A; no longer LED10.A
- net LED8: now also LED10.A; no longer LED9.A
Changed lines of the file:
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@@
 </segment>
 <segment>
-<pinref part="LED10" gate="G$1" pin="A"/>
-<wire x1="-774.7" y1="-200.66" x2="-772.16" y2="-200.66" width="0.1524" layer="91"/>
-<label x="-774.7" y="-200.66" size="1.27" layer="95" font="vector" ratio="10" rot="R180" xref="yes"/>
+<pinref part="LED9" gate="G$1" pin="A"/>
+<wire x1="-774.7" y1="-193.04" x2="-772.16" y2="-193.04" width="0.1524" layer="91"/>
+<label x="-774.7" y="-193.04" size="1.27" layer="95" font="vector" ratio="10" rot="R180" xref="yes"/>
 </segment>
 </net>
@@
 </segment>
 <segment>
-<pinref part="LED9" gate="G$1" pin="A"/>
-<wire x1="-774.7" y1="-193.04" x2="-772.16" y2="-193.04" width="0.1524" layer="91"/>
-<label x="-774.7" y="-193.04" size="1.27" layer="95" font="vector" ratio="10" rot="R180" xref="yes"/>
+<pinref part="LED10" gate="G$1" pin="A"/>
+<wire x1="-774.7" y1="-200.66" x2="-772.16" y2="-200.66" width="0.1524" layer="91"/>
+<label x="-774.7" y="-200.66" size="1.27" layer="95" font="vector" ratio="10" rot="R180" xref="yes"/>
 </segment>
 </net>

Commit message: Almost done with heart necklace
Parts:
- removed BATT1: 3V/CR2032, PiB:BATTERY_CELL_COINCELL-CR2032-20MM_PTH
- added AVR_ISP1: (no value), PiB_connectors:AVR_SPI_PRG_6NS-PAD
- added BATT2: BR-1225/3V/48mAh, PiB_batteries:BATTERY_COIN-CELL_SMD_3V_12.5MM
Connections:
- removed net N$14: MCU1.(PCINT11/!RESET!/DW/D11)PB3
- new net !RESET: AVR_ISP1.5, MCU1.(PCINT11/!RESET!/DW/D11)PB3
- new net VCC: AVR_ISP1.2
- net GND: now also AVR_ISP1.6, BATT2.-; no longer BATT1.-
- net LED10: now also AVR_ISP1.4
- net LED4: now also AVR_ISP1.1
- net LED6: now also AVR_ISP1.3
- net VBATT: now also BATT2.+; no longer BATT1.+
Other:
- note added: "!RESET"
- note added: "MISO"
- note added: "MOSI"
- note added: "SCK"
Changed lines of the file:
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@@
 <?xml version="1.0" encoding="utf-8"?>
 <!DOCTYPE eagle SYSTEM "eagle.dtd">
-<eagle version="8.4.1">
+<eagle version="8.5.0">
 <drawing>
 <settings>
-<setting alwaysvectorfont="no"/>
+<setting alwaysvectorfont="yes"/>
 <setting keepoldvectorfont="yes"/>
 <setting verticaltext="up"/>
 </settings>
-<grid distance="0.1" unitdist="inch" unit="inch" style="lines" multiple="1" display="no" altdistance="0.01" altunitdist="inch" altunit="inch"/>
+<grid distance="0.1" unitdist="inch" unit="inch" style="lines" multiple="1" display="yes" altdistance="0.01" altunitdist="inch" altunit="inch"/>
 <layers>
 <layer number="1" name="Top" color="4" fill="10" visible="no" active="no"/>
@@
 <layer number="59" name="tCarbon" color="7" fill="1" visible="no" active="no"/>
 <layer number="60" name="bCarbon" color="7" fill="1" visible="no" active="no"/>
+<layer number="88" name="SimResults" color="9" fill="1" visible="yes" active="yes"/>
+<layer number="89" name="SimProbes" color="9" fill="1" visible="yes" active="yes"/>
 <layer number="90" name="Modules" color="5" fill="1" visible="yes" active="yes"/>
 <layer number="91" name="Nets" color="2" fill="1" visible="yes" active="yes"/>
@@
 <part name="SW1" library="PiB_switches" deviceset="SWITCH_SPDT" device="_RA_SMD_300MA-4V_6.7L-2.6W" value="300mA/4V"/>
 <part name="GND1" library="PiB_power_symbols" deviceset="GND" device=""/>
-<part name="BATT1" library="PiB" deviceset="BATTERY_CELL" device="_COINCELL-CR2032-20MM_PTH" value="3V/CR2032"/>
 <part name="GND3" library="PiB_power_symbols" deviceset="GND" device=""/>
+<part name="BATT2" library="PiB_batteries" deviceset="BATTERY_COIN-CELL" device="_SMD_3V_12.5MM" value="BR-1225/3V/48mAh"/>
+<part name="AVR_ISP1" library="PiB_connectors" deviceset="AVR_SPI_PRG_6" device="NS-PAD"/>
+<part name="SUPPLY1" library="PiB_power_symbols" deviceset="GND" device=""/>
+<part name="SUPPLY2" library="PiB_power_symbols" deviceset="VCC" device=""/>
 </parts>
 <sheets>
@@
 <plain>
 <text x="-812.8" y="-177.8" size="1.27" layer="97" font="vector" ratio="10">NC</text>
-<text x="-812.8" y="-185.42" size="1.27" layer="97" font="vector" ratio="10">NC</text>
 <wire x1="-787.4" y1="-124.46" x2="-787.4" y2="-213.36" width="0.1524" layer="97" style="shortdash"/>
 <wire x1="-787.4" y1="-213.36" x2="-741.68" y2="-213.36" width="0.1524" layer="97" style="shortdash"/>
@@
 <text x="-853.44" y="-142.24" size="7.62" layer="97" font="vector" ratio="20" align="bottom-center">ATTINY84</text>
 <text x="-896.62" y="-152.4" size="1.27" layer="97" font="vector" ratio="10" rot="MR0">NC</text>
+<text x="-800.1" y="-165.1" size="1.27" layer="91" font="vector" ratio="10">SCK</text>
+<text x="-800.1" y="-167.64" size="1.27" layer="91" font="vector" ratio="10">MISO</text>
+<text x="-800.1" y="-170.18" size="1.27" layer="91" font="vector" ratio="10">MOSI</text>
+<text x="-800.1" y="-185.42" size="1.27" layer="91" font="vector" ratio="10">!RESET</text>
 </plain>
 <instances>
@@
 <instance part="SW1" gate="G$1" x="-891.54" y="-154.94" rot="R180"/>
 <instance part="GND1" gate="GND" x="-749.3" y="-205.74"/>
-<instance part="BATT1" gate="G$1" x="-904.24" y="-162.56"/>
 <instance part="GND3" gate="GND" x="-886.46" y="-190.5"/>
+<instance part="BATT2" gate="G$1" x="-904.24" y="-162.56"/>
+<instance part="AVR_ISP1" gate="G$1" x="-853.44" y="-218.44"/>
+<instance part="SUPPLY1" gate="GND" x="-843.28" y="-226.06"/>
+<instance part="SUPPLY2" gate="VCC" x="-843.28" y="-213.36"/>
 </instances>
 <busses>
@@
 <pinref part="GND2" gate="GND" pin="GND"/>
 <wire x1="-904.24" y1="-167.64" x2="-904.24" y2="-170.18" width="0.1524" layer="91"/>
-<pinref part="BATT1" gate="G$1" pin="-"/>
+<pinref part="BATT2" gate="G$1" pin="-"/>
 </segment>
 <segment>
@@
 <wire x1="-886.46" y1="-185.42" x2="-883.92" y2="-185.42" width="0.1524" layer="91"/>
 </segment>
+<segment>
+<pinref part="AVR_ISP1" gate="G$1" pin="6"/>
+<wire x1="-845.82" y1="-220.98" x2="-843.28" y2="-220.98" width="0.1524" layer="91"/>
+<wire x1="-843.28" y1="-220.98" x2="-843.28" y2="-223.52" width="0.1524" layer="91"/>
+<pinref part="SUPPLY1" gate="GND" pin="GND"/>
+</segment>
 </net>
 <net name="VBATT" class="0">
 <segment>
-<pinref part="BATT1" gate="G$1" pin="+"/>
 <wire x1="-904.24" y1="-160.02" x2="-904.24" y2="-157.48" width="0.1524" layer="91"/>
 <pinref part="SW1" gate="G$1" pin="1"/>
 <wire x1="-896.62" y1="-157.48" x2="-904.24" y2="-157.48" width="0.1524" layer="91"/>
+<pinref part="BATT2" gate="G$1" pin="+"/>
 </segment>
 </net>
@@
 <label x="-774.7" y="-170.18" size="1.27" layer="95" font="vector" ratio="10" rot="R180" xref="yes"/>
 </segment>
+<segment>
+<pinref part="AVR_ISP1" gate="G$1" pin="1"/>
+<wire x1="-863.6" y1="-215.9" x2="-861.06" y2="-215.9" width="0.1524" layer="91"/>
+<label x="-863.6" y="-215.9" size="1.27" layer="95" font="vector" ratio="10" rot="R180" xref="yes"/>
+</segment>
 </net>
 <net name="LED5" class="0">
@@
 <label x="-774.7" y="-162.56" size="1.27" layer="95" font="vector" ratio="10" rot="R180" xref="yes"/>
 </segment>
+<segment>
+<pinref part="AVR_ISP1" gate="G$1" pin="3"/>
+<wire x1="-861.06" y1="-218.44" x2="-863.6" y2="-218.44" width="0.1524" layer="91"/>
+<label x="-863.6" y="-218.44" size="1.27" layer="95" font="vector" ratio="10" rot="R180" xref="yes"/>
+</segment>
 </net>
 <net name="LED10" class="0">
@@
 <label x="-774.7" y="-177.8" size="1.27" layer="95" font="vector" ratio="10" rot="R180" xref="yes"/>
 </segment>
+<segment>
+<pinref part="AVR_ISP1" gate="G$1" pin="4"/>
+<wire x1="-843.28" y1="-218.44" x2="-845.82" y2="-218.44" width="0.1524" layer="91"/>
+<label x="-843.28" y="-218.44" size="1.27" layer="95" font="vector" ratio="10" xref="yes"/>
+</segment>
 </net>
 <net name="LED8" class="0">
@@
 </segment>
 </net>
-<net name="N$14" class="0">
+<net name="!RESET" class="0">
 <segment>
 <pinref part="MCU1" gate="G$1" pin="(PCINT11/!RESET!/DW/D11)PB3"/>
+<wire x1="-810.26" y1="-185.42" x2="-812.8" y2="-185.42" width="0.1524" layer="91"/>
+<label x="-810.26" y="-185.42" size="1.27" layer="95" font="vector" ratio="10" xref="yes"/>
+</segment>
+<segment>
+<pinref part="AVR_ISP1" gate="G$1" pin="5"/>
+<wire x1="-863.6" y1="-220.98" x2="-861.06" y2="-220.98" width="0.1524" layer="91"/>
+<label x="-863.6" y="-220.98" size="1.27" layer="95" font="vector" ratio="10" rot="R180" xref="yes"/>
 </segment>
 </net>
@@
 </segment>
 </net>
+<net name="VCC" class="0">
+<segment>
+<pinref part="AVR_ISP1" gate="G$1" pin="2"/>
+<wire x1="-843.28" y1="-215.9" x2="-845.82" y2="-215.9" width="0.1524" layer="91"/>
+<wire x1="-843.28" y1="-215.9" x2="-843.28" y2="-213.36" width="0.1524" layer="91"/>
+<pinref part="SUPPLY2" gate="VCC" pin="VCC"/>
+</segment>
+</net>

Commit message: Rev 1: Heart Necklace complete
Parts:
- removed AVR_ISP1: (no value), PiB_connectors:AVR_SPI_PRG_6NS-PAD
- LED1, LED10, LED2, LED3, LED4, LED5, LED6, LED7, LED8, LED9: device PiB_leds:LED_SMD-0805_DISCRETE_BLUE -> PiB_leds:LED_SMD-0805_DISCRETE_NO-COLOR_NO-SILK
- MCU1: device PiB_ic_microcontrollers:ATTINY84_SO-14 -> PiB_ic_microcontrollers:ATTINY84_SO-14_NO-SILK
Connections:
- removed net VCC: AVR_ISP1.2
- net !RESET: no longer AVR_ISP1.5
- net GND: no longer AVR_ISP1.6
- net LED10: no longer AVR_ISP1.4
- net LED4: no longer AVR_ISP1.1
- net LED6: no longer AVR_ISP1.3
Changed lines of the file:
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@@
 <setting verticaltext="up"/>
 </settings>
-<grid distance="0.1" unitdist="inch" unit="inch" style="lines" multiple="1" display="yes" altdistance="0.01" altunitdist="inch" altunit="inch"/>
+<grid distance="0.1" unitdist="inch" unit="inch" style="lines" multiple="1" display="no" altdistance="0.01" altunitdist="inch" altunit="inch"/>
 <layers>
 <layer number="1" name="Top" color="4" fill="10" visible="no" active="no"/>
@@
 </classes>
 <parts>
-<part name="LED3" library="PiB_leds" deviceset="LED" device="_SMD-0805_DISCRETE_BLUE" value="BLUE"/>
-<part name="LED2" library="PiB_leds" deviceset="LED" device="_SMD-0805_DISCRETE_BLUE" value="BLUE"/>
-<part name="LED1" library="PiB_leds" deviceset="LED" device="_SMD-0805_DISCRETE_BLUE" value="BLUE"/>
-<part name="LED10" library="PiB_leds" deviceset="LED" device="_SMD-0805_DISCRETE_BLUE" value="BLUE"/>
-<part name="LED9" library="PiB_leds" deviceset="LED" device="_SMD-0805_DISCRETE_BLUE" value="BLUE"/>
-<part name="LED8" library="PiB_leds" deviceset="LED" device="_SMD-0805_DISCRETE_BLUE" value="BLUE"/>
-<part name="LED7" library="PiB_leds" deviceset="LED" device="_SMD-0805_DISCRETE_BLUE" value="BLUE"/>
-<part name="LED6" library="PiB_leds" deviceset="LED" device="_SMD-0805_DISCRETE_BLUE" value="BLUE"/>
-<part name="LED5" library="PiB_leds" deviceset="LED" device="_SMD-0805_DISCRETE_BLUE" value="BLUE"/>
-<part name="LED4" library="PiB_leds" deviceset="LED" device="_SMD-0805_DISCRETE_BLUE" value="BLUE"/>
+<part name="LED3" library="PiB_leds" deviceset="LED" device="_SMD-0805_DISCRETE_NO-COLOR_NO-SILK" value="BLUE"/>
+<part name="LED2" library="PiB_leds" deviceset="LED" device="_SMD-0805_DISCRETE_NO-COLOR_NO-SILK" value="BLUE"/>
+<part name="LED1" library="PiB_leds" deviceset="LED" device="_SMD-0805_DISCRETE_NO-COLOR_NO-SILK" value="BLUE"/>
+<part name="LED10" library="PiB_leds" deviceset="LED" device="_SMD-0805_DISCRETE_NO-COLOR_NO-SILK" value="BLUE"/>
+<part name="LED9" library="PiB_leds" deviceset="LED" device="_SMD-0805_DISCRETE_NO-COLOR_NO-SILK" value="BLUE"/>
+<part name="LED8" library="PiB_leds" deviceset="LED" device="_SMD-0805_DISCRETE_NO-COLOR_NO-SILK" value="BLUE"/>
+<part name="LED7" library="PiB_leds" deviceset="LED" device="_SMD-0805_DISCRETE_NO-COLOR_NO-SILK" value="BLUE"/>
+<part name="LED6" library="PiB_leds" deviceset="LED" device="_SMD-0805_DISCRETE_NO-COLOR_NO-SILK" value="BLUE"/>
+<part name="LED5" library="PiB_leds" deviceset="LED" device="_SMD-0805_DISCRETE_NO-COLOR_NO-SILK" value="BLUE"/>
+<part name="LED4" library="PiB_leds" deviceset="LED" device="_SMD-0805_DISCRETE_NO-COLOR_NO-SILK" value="BLUE"/>
 <part name="R3" library="PiB_resistors" deviceset="1KΩ" device="_SMD-0805_1/8W-5%" value="1KΩ"/>
 <part name="R2" library="PiB_resistors" deviceset="1KΩ" device="_SMD-0805_1/8W-5%" value="1KΩ"/>
@@
 <part name="R4" library="PiB_resistors" deviceset="1KΩ" device="_SMD-0805_1/8W-5%" value="1KΩ"/>
 <part name="GND2" library="PiB_power_symbols" deviceset="GND" device=""/>
-<part name="MCU1" library="PiB_ic_microcontrollers" deviceset="ATTINY84" device="_SO-14" value="ATTINY84"/>
+<part name="MCU1" library="PiB_ic_microcontrollers" deviceset="ATTINY84" device="_SO-14_NO-SILK" value="ATTINY84"/>
 <part name="SW1" library="PiB_switches" deviceset="SWITCH_SPDT" device="_RA_SMD_300MA-4V_6.7L-2.6W" value="300mA/4V"/>
 <part name="GND1" library="PiB_power_symbols" deviceset="GND" device=""/>
 <part name="GND3" library="PiB_power_symbols" deviceset="GND" device=""/>
 <part name="BATT2" library="PiB_batteries" deviceset="BATTERY_COIN-CELL" device="_SMD_3V_12.5MM" value="BR-1225/3V/48mAh"/>
-<part name="AVR_ISP1" library="PiB_connectors" deviceset="AVR_SPI_PRG_6" device="NS-PAD"/>
-<part name="SUPPLY1" library="PiB_power_symbols" deviceset="GND" device=""/>
-<part name="SUPPLY2" library="PiB_power_symbols" deviceset="VCC" device=""/>
 </parts>
 <sheets>
@@
 <instance part="GND3" gate="GND" x="-886.46" y="-190.5"/>
 <instance part="BATT2" gate="G$1" x="-904.24" y="-162.56"/>
-<instance part="AVR_ISP1" gate="G$1" x="-853.44" y="-218.44"/>
-<instance part="SUPPLY1" gate="GND" x="-843.28" y="-226.06"/>
-<instance part="SUPPLY2" gate="VCC" x="-843.28" y="-213.36"/>
 </instances>
 <busses>
@@
 <wire x1="-886.46" y1="-185.42" x2="-883.92" y2="-185.42" width="0.1524" layer="91"/>
 </segment>
-<segment>
-<pinref part="AVR_ISP1" gate="G$1" pin="6"/>
-<wire x1="-845.82" y1="-220.98" x2="-843.28" y2="-220.98" width="0.1524" layer="91"/>
-<wire x1="-843.28" y1="-220.98" x2="-843.28" y2="-223.52" width="0.1524" layer="91"/>
-<pinref part="SUPPLY1" gate="GND" pin="GND"/>
-</segment>
 </net>
 <net name="VBATT" class="0">
@@
 <label x="-774.7" y="-170.18" size="1.27" layer="95" font="vector" ratio="10" rot="R180" xref="yes"/>
 </segment>
-<segment>
-<pinref part="AVR_ISP1" gate="G$1" pin="1"/>
-<wire x1="-863.6" y1="-215.9" x2="-861.06" y2="-215.9" width="0.1524" layer="91"/>
-<label x="-863.6" y="-215.9" size="1.27" layer="95" font="vector" ratio="10" rot="R180" xref="yes"/>
-</segment>
 </net>
 <net name="LED5" class="0">
@@
 <label x="-774.7" y="-162.56" size="1.27" layer="95" font="vector" ratio="10" rot="R180" xref="yes"/>
 </segment>
-<segment>
-<pinref part="AVR_ISP1" gate="G$1" pin="3"/>
-<wire x1="-861.06" y1="-218.44" x2="-863.6" y2="-218.44" width="0.1524" layer="91"/>
-<label x="-863.6" y="-218.44" size="1.27" layer="95" font="vector" ratio="10" rot="R180" xref="yes"/>
-</segment>
 </net>
 <net name="LED10" class="0">
@@
 <label x="-774.7" y="-177.8" size="1.27" layer="95" font="vector" ratio="10" rot="R180" xref="yes"/>
 </segment>
-<segment>
-<pinref part="AVR_ISP1" gate="G$1" pin="4"/>
-<wire x1="-843.28" y1="-218.44" x2="-845.82" y2="-218.44" width="0.1524" layer="91"/>
-<label x="-843.28" y="-218.44" size="1.27" layer="95" font="vector" ratio="10" xref="yes"/>
-</segment>
 </net>
 <net name="LED8" class="0">
@@
 <label x="-810.26" y="-185.42" size="1.27" layer="95" font="vector" ratio="10" xref="yes"/>
 </segment>
-<segment>
-<pinref part="AVR_ISP1" gate="G$1" pin="5"/>
-<wire x1="-863.6" y1="-220.98" x2="-861.06" y2="-220.98" width="0.1524" layer="91"/>
-<label x="-863.6" y="-220.98" size="1.27" layer="95" font="vector" ratio="10" rot="R180" xref="yes"/>
-</segment>
 </net>
 <net name="N$17" class="0">
@@
 </segment>
 </net>
-<net name="VCC" class="0">
-<segment>
-<pinref part="AVR_ISP1" gate="G$1" pin="2"/>
-<wire x1="-843.28" y1="-215.9" x2="-845.82" y2="-215.9" width="0.1524" layer="91"/>
-<wire x1="-843.28" y1="-215.9" x2="-843.28" y2="-213.36" width="0.1524" layer="91"/>
-<pinref part="SUPPLY2" gate="VCC" pin="VCC"/>
-</segment>
-</net>

Commit message: changes
Parts:
- removed BATT2: BR-1225/3V/48mAh, PiB_batteries:BATTERY_COIN-CELL_SMD_3V_12.5MM
- added BATT1: (no value), PiB_batteries:BATTERY_COIN-CELL_SMD_3V_20MM
- added C1, C2: 10uF/10V, PiB_capacitors:10UF_CER_SMD-0402_10V-20%
- MCU1: value ATTINY84 -> ATTiny84
Connections:
- net GND: now also BATT1.-, C1.2, C2.2; no longer BATT2.-
- net N$11: now also C1.1, C2.1, SW1.3; no longer SW1.2
- net VBATT: now also BATT1.+, SW1.2; no longer BATT2.+, SW1.1
Other:
- moved on the sheet: SW1
Changed lines of the file:
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@@
 <part name="R4" library="PiB_resistors" deviceset="1KΩ" device="_SMD-0805_1/8W-5%" value="1KΩ"/>
 <part name="GND2" library="PiB_power_symbols" deviceset="GND" device=""/>
-<part name="MCU1" library="PiB_ic_microcontrollers" deviceset="ATTINY84" device="_SO-14_NO-SILK" value="ATTINY84"/>
+<part name="MCU1" library="PiB_ic_microcontrollers" deviceset="ATTINY84" device="_SO-14_NO-SILK" value="ATTiny84"/>
 <part name="SW1" library="PiB_switches" deviceset="SWITCH_SPDT" device="_RA_SMD_300MA-4V_6.7L-2.6W" value="300mA/4V"/>
 <part name="GND1" library="PiB_power_symbols" deviceset="GND" device=""/>
 <part name="GND3" library="PiB_power_symbols" deviceset="GND" device=""/>
-<part name="BATT2" library="PiB_batteries" deviceset="BATTERY_COIN-CELL" device="_SMD_3V_12.5MM" value="BR-1225/3V/48mAh"/>
+<part name="BATT1" library="PiB_batteries" deviceset="BATTERY_COIN-CELL" device="_SMD_3V_20MM"/>
+<part name="C1" library="PiB_capacitors" deviceset="10UF" device="_CER_SMD-0402_10V-20%" value="10uF/10V"/>
+<part name="GND4" library="PiB_power_symbols" deviceset="GND" device=""/>
+<part name="C2" library="PiB_capacitors" deviceset="10UF" device="_CER_SMD-0402_10V-20%" value="10uF/10V"/>
+<part name="GND5" library="PiB_power_symbols" deviceset="GND" device=""/>
 </parts>
 <sheets>
@@
 <wire x1="-741.68" y1="-124.46" x2="-787.4" y2="-124.46" width="0.1524" layer="97" style="shortdash"/>
 <text x="-762" y="-121.92" size="7.62" layer="97" font="vector" ratio="20" align="bottom-center">LEDS</text>
-<wire x1="-914.4" y1="-144.78" x2="-914.4" y2="-198.12" width="0.1524" layer="97" style="shortdash"/>
-<wire x1="-914.4" y1="-198.12" x2="-797.56" y2="-198.12" width="0.1524" layer="97" style="shortdash"/>
+<wire x1="-924.56" y1="-144.78" x2="-924.56" y2="-198.12" width="0.1524" layer="97" style="shortdash"/>
+<wire x1="-924.56" y1="-198.12" x2="-797.56" y2="-198.12" width="0.1524" layer="97" style="shortdash"/>
 <wire x1="-797.56" y1="-198.12" x2="-797.56" y2="-144.78" width="0.1524" layer="97" style="shortdash"/>
-<wire x1="-797.56" y1="-144.78" x2="-914.4" y2="-144.78" width="0.1524" layer="97" style="shortdash"/>
+<wire x1="-797.56" y1="-144.78" x2="-924.56" y2="-144.78" width="0.1524" layer="97" style="shortdash"/>
 <text x="-853.44" y="-142.24" size="7.62" layer="97" font="vector" ratio="20" align="bottom-center">ATTINY84</text>
-<text x="-896.62" y="-152.4" size="1.27" layer="97" font="vector" ratio="10" rot="MR0">NC</text>
+<text x="-906.78" y="-152.4" size="1.27" layer="97" font="vector" ratio="10" rot="MR0">NC</text>
 <text x="-800.1" y="-165.1" size="1.27" layer="91" font="vector" ratio="10">SCK</text>
 <text x="-800.1" y="-167.64" size="1.27" layer="91" font="vector" ratio="10">MISO</text>
@@
 <instance part="R5" gate="G$1" x="-756.92" y="-162.56" rot="MR0"/>
 <instance part="R4" gate="G$1" x="-756.92" y="-154.94" rot="MR0"/>
-<instance part="GND2" gate="GND" x="-904.24" y="-172.72"/>
+<instance part="GND2" gate="GND" x="-914.4" y="-172.72"/>
 <instance part="MCU1" gate="G$1" x="-848.36" y="-170.18"/>
-<instance part="SW1" gate="G$1" x="-891.54" y="-154.94" rot="R180"/>
+<instance part="SW1" gate="G$1" x="-904.24" y="-152.4"/>
 <instance part="GND1" gate="GND" x="-749.3" y="-205.74"/>
 <instance part="GND3" gate="GND" x="-886.46" y="-190.5"/>
-<instance part="BATT2" gate="G$1" x="-904.24" y="-162.56"/>
+<instance part="BATT1" gate="G$1" x="-914.4" y="-162.56"/>
+<instance part="C1" gate="G$1" x="-886.46" y="-157.48"/>
+<instance part="GND4" gate="GND" x="-886.46" y="-165.1"/>
+<instance part="C2" gate="G$1" x="-894.08" y="-157.48"/>
+<instance part="GND5" gate="GND" x="-894.08" y="-165.1"/>
 </instances>
 <busses>
@@
 <segment>
 <pinref part="GND2" gate="GND" pin="GND"/>
-<wire x1="-904.24" y1="-167.64" x2="-904.24" y2="-170.18" width="0.1524" layer="91"/>
-<pinref part="BATT2" gate="G$1" pin="-"/>
+<wire x1="-914.4" y1="-167.64" x2="-914.4" y2="-170.18" width="0.1524" layer="91"/>
+<pinref part="BATT1" gate="G$1" pin="-"/>
 </segment>
 <segment>
@@
 <wire x1="-886.46" y1="-185.42" x2="-883.92" y2="-185.42" width="0.1524" layer="91"/>
 </segment>
+<segment>
+<pinref part="C1" gate="G$1" pin="2"/>
+<pinref part="GND4" gate="GND" pin="GND"/>
+</segment>
+<segment>
+<pinref part="C2" gate="G$1" pin="2"/>
+<pinref part="GND5" gate="GND" pin="GND"/>
+</segment>
 </net>
 <net name="VBATT" class="0">
 <segment>
-<wire x1="-904.24" y1="-160.02" x2="-904.24" y2="-157.48" width="0.1524" layer="91"/>
-<pinref part="SW1" gate="G$1" pin="1"/>
-<wire x1="-896.62" y1="-157.48" x2="-904.24" y2="-157.48" width="0.1524" layer="91"/>
-<pinref part="BATT2" gate="G$1" pin="+"/>
+<wire x1="-914.4" y1="-160.02" x2="-914.4" y2="-152.4" width="0.1524" layer="91"/>
+<pinref part="BATT1" gate="G$1" pin="+"/>
+<pinref part="SW1" gate="G$1" pin="2"/>
+<wire x1="-906.78" y1="-152.4" x2="-914.4" y2="-152.4" width="0.1524" layer="91"/>
 </segment>
 </net>
@@
 <net name="N$11" class="0">
 <segment>
-<pinref part="SW1" gate="G$1" pin="2"/>
+<pinref part="SW1" gate="G$1" pin="3"/>
 <pinref part="MCU1" gate="G$1" pin="VCC"/>
-<wire x1="-889" y1="-154.94" x2="-883.92" y2="-154.94" width="0.1524" layer="91"/>
-</segment>
-</net>
+<wire x1="-899.16" y1="-154.94" x2="-894.08" y2="-154.94" width="0.1524" layer="91"/>
+<pinref part="C1" gate="G$1" pin="1"/>
+<wire x1="-894.08" y1="-154.94" x2="-886.46" y2="-154.94" width="0.1524" layer="91"/>
+<wire x1="-886.46" y1="-154.94" x2="-883.92" y2="-154.94" width="0.1524" layer="91"/>
+<junction x="-886.46" y="-154.94"/>
+<pinref part="C2" gate="G$1" pin="1"/>
+<junction x="-894.08" y="-154.94"/>
+</segment>
+</net>
