File: ecad/heart_necklace.brd (EAGLE design)
At the start: 36.5 x 34 mm, 25 parts, among them SW1 300mA/4V

Commit message: Initialize heart necklace repo?
Parts:
- BATT1: value 3V/225mAh -> 225mAh/3V
- C1, C2: value 10uF/10V -> 10uF/6.3V; device PiB_capacitors:_CER_SMD_0402 -> PiB_capacitors:CAPC1005X55_SMD-0402
- LED1, LED10, LED2, LED3, LED4, LED5, LED6, LED7, LED8, LED9: device PiB_leds:LED_SMD-805_NO-SILK -> PiB_leds:LEDC2012X120
- MCU1: value ATTiny84 -> ATtiny84; device PiB_ic_microcontrollers:SO-14_NO-SILK -> PiB_ic_microcontrollers:SOIC127P599X175-14_SOIC-14_NO-SILK
- moved C2 0.13 mm to (-11.3, 25.5)
Other:
- board text added: "Rev 3"
- board text removed: "Rev 2"
