File: ecad/heart_necklace.sch (EAGLE design)
At the start: 25 parts, among them SW1 300mA/4V

Commit message: Initialize heart necklace repo?
Parts:
- BATT1: value 3V/225mAh -> 225mAh/3V
- C1, C2: value 10uF/10V -> 10uF/6.3V; device PiB_capacitors:10UF_CER_SMD-0402_10V-20% -> PiB_capacitors:10UF_CER_SMD-0402_6.3V-20%
- LED1, LED10, LED2, LED3, LED4, LED5, LED6, LED7, LED8, LED9: device PiB_leds:LED_SMD-0805_DISCRETE_NO-COLOR_NO-SILK -> PiB_leds:LED_SMD-0805_DISCRETE_BLUE
- MCU1: value ATTiny84 -> ATtiny84; device PiB_ic_microcontrollers:ATTINY84_SO-14_NO-SILK -> PiB_ic_microcontrollers:ATTINY84_SOIC-14_NO_SILK
Connections:
- net N$11: now also SW1.S2; no longer SW1.3
- net VBATT: now also SW1.P; no longer SW1.2
Changed lines of the file:
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@@
 <?xml version="1.0" encoding="utf-8"?>
 <!DOCTYPE eagle SYSTEM "eagle.dtd">
-<eagle version="8.5.0">
+<eagle version="9.0.1">
 <drawing>
 <settings>
@@
 </classes>
 <parts>
-<part name="LED3" library="PiB_leds" deviceset="LED" device="_SMD-0805_DISCRETE_NO-COLOR_NO-SILK" value="BLUE"/>
-<part name="LED2" library="PiB_leds" deviceset="LED" device="_SMD-0805_DISCRETE_NO-COLOR_NO-SILK" value="BLUE"/>
-<part name="LED1" library="PiB_leds" deviceset="LED" device="_SMD-0805_DISCRETE_NO-COLOR_NO-SILK" value="BLUE"/>
-<part name="LED10" library="PiB_leds" deviceset="LED" device="_SMD-0805_DISCRETE_NO-COLOR_NO-SILK" value="BLUE"/>
-<part name="LED9" library="PiB_leds" deviceset="LED" device="_SMD-0805_DISCRETE_NO-COLOR_NO-SILK" value="BLUE"/>
-<part name="LED8" library="PiB_leds" deviceset="LED" device="_SMD-0805_DISCRETE_NO-COLOR_NO-SILK" value="BLUE"/>
-<part name="LED7" library="PiB_leds" deviceset="LED" device="_SMD-0805_DISCRETE_NO-COLOR_NO-SILK" value="BLUE"/>
-<part name="LED6" library="PiB_leds" deviceset="LED" device="_SMD-0805_DISCRETE_NO-COLOR_NO-SILK" value="BLUE"/>
-<part name="LED5" library="PiB_leds" deviceset="LED" device="_SMD-0805_DISCRETE_NO-COLOR_NO-SILK" value="BLUE"/>
-<part name="LED4" library="PiB_leds" deviceset="LED" device="_SMD-0805_DISCRETE_NO-COLOR_NO-SILK" value="BLUE"/>
-<part name="R3" library="PiB_resistors" deviceset="1KΩ" device="_SMD-0805_1/8W-5%" value="1KΩ"/>
-<part name="R2" library="PiB_resistors" deviceset="1KΩ" device="_SMD-0805_1/8W-5%" value="1KΩ"/>
-<part name="R1" library="PiB_resistors" deviceset="1KΩ" device="_SMD-0805_1/8W-5%" value="1KΩ"/>
-<part name="R10" library="PiB_resistors" deviceset="1KΩ" device="_SMD-0805_1/8W-5%" value="1KΩ"/>
-<part name="R9" library="PiB_resistors" deviceset="1KΩ" device="_SMD-0805_1/8W-5%" value="1KΩ"/>
-<part name="R8" library="PiB_resistors" deviceset="1KΩ" device="_SMD-0805_1/8W-5%" value="1KΩ"/>
-<part name="R7" library="PiB_resistors" deviceset="1KΩ" device="_SMD-0805_1/8W-5%" value="1KΩ"/>
-<part name="R6" library="PiB_resistors" deviceset="1KΩ" device="_SMD-0805_1/8W-5%" value="1KΩ"/>
-<part name="R5" library="PiB_resistors" deviceset="1KΩ" device="_SMD-0805_1/8W-5%" value="1KΩ"/>
-<part name="R4" library="PiB_resistors" deviceset="1KΩ" device="_SMD-0805_1/8W-5%" value="1KΩ"/>
+<part name="LED3" library="PiB_leds" deviceset="LED" device="_SMD-0805_DISCRETE_BLUE" package3d_urn="urn:adsk.eagle:package:2966314/1" value="BLUE"/>
+<part name="LED2" library="PiB_leds" deviceset="LED" device="_SMD-0805_DISCRETE_BLUE" package3d_urn="urn:adsk.eagle:package:2966314/1" value="BLUE"/>
+<part name="LED1" library="PiB_leds" deviceset="LED" device="_SMD-0805_DISCRETE_BLUE" package3d_urn="urn:adsk.eagle:package:2966314/1" value="BLUE"/>
+<part name="LED10" library="PiB_leds" deviceset="LED" device="_SMD-0805_DISCRETE_BLUE" package3d_urn="urn:adsk.eagle:package:2966314/1" value="BLUE"/>
+<part name="LED9" library="PiB_leds" deviceset="LED" device="_SMD-0805_DISCRETE_BLUE" package3d_urn="urn:adsk.eagle:package:2966314/1" value="BLUE"/>
+<part name="LED8" library="PiB_leds" deviceset="LED" device="_SMD-0805_DISCRETE_BLUE" package3d_urn="urn:adsk.eagle:package:2966314/1" value="BLUE"/>
+<part name="LED7" library="PiB_leds" deviceset="LED" device="_SMD-0805_DISCRETE_BLUE" package3d_urn="urn:adsk.eagle:package:2966314/1" value="BLUE"/>
+<part name="LED6" library="PiB_leds" deviceset="LED" device="_SMD-0805_DISCRETE_BLUE" package3d_urn="urn:adsk.eagle:package:2966314/1" value="BLUE"/>
+<part name="LED5" library="PiB_leds" deviceset="LED" device="_SMD-0805_DISCRETE_BLUE" package3d_urn="urn:adsk.eagle:package:2966314/1" value="BLUE"/>
+<part name="LED4" library="PiB_leds" deviceset="LED" device="_SMD-0805_DISCRETE_BLUE" package3d_urn="urn:adsk.eagle:package:2966314/1" value="BLUE"/>
+<part name="R3" library="PiB_resistors" deviceset="1KΩ" device="_SMD-0805_1/8W-5%" package3d_urn="urn:adsk.eagle:package:2749855/3" value="1KΩ"/>
+<part name="R2" library="PiB_resistors" deviceset="1KΩ" device="_SMD-0805_1/8W-5%" package3d_urn="urn:adsk.eagle:package:2749855/3" value="1KΩ"/>
+<part name="R1" library="PiB_resistors" deviceset="1KΩ" device="_SMD-0805_1/8W-5%" package3d_urn="urn:adsk.eagle:package:2749855/3" value="1KΩ"/>
+<part name="R10" library="PiB_resistors" deviceset="1KΩ" device="_SMD-0805_1/8W-5%" package3d_urn="urn:adsk.eagle:package:2749855/3" value="1KΩ"/>
+<part name="R9" library="PiB_resistors" deviceset="1KΩ" device="_SMD-0805_1/8W-5%" package3d_urn="urn:adsk.eagle:package:2749855/3" value="1KΩ"/>
+<part name="R8" library="PiB_resistors" deviceset="1KΩ" device="_SMD-0805_1/8W-5%" package3d_urn="urn:adsk.eagle:package:2749855/3" value="1KΩ"/>
+<part name="R7" library="PiB_resistors" deviceset="1KΩ" device="_SMD-0805_1/8W-5%" package3d_urn="urn:adsk.eagle:package:2749855/3" value="1KΩ"/>
+<part name="R6" library="PiB_resistors" deviceset="1KΩ" device="_SMD-0805_1/8W-5%" package3d_urn="urn:adsk.eagle:package:2749855/3" value="1KΩ"/>
+<part name="R5" library="PiB_resistors" deviceset="1KΩ" device="_SMD-0805_1/8W-5%" package3d_urn="urn:adsk.eagle:package:2749855/3" value="1KΩ"/>
+<part name="R4" library="PiB_resistors" deviceset="1KΩ" device="_SMD-0805_1/8W-5%" package3d_urn="urn:adsk.eagle:package:2749855/3" value="1KΩ"/>
 <part name="GND2" library="PiB_power_symbols" deviceset="GND" device=""/>
-<part name="MCU1" library="PiB_ic_microcontrollers" deviceset="ATTINY84" device="_SO-14_NO-SILK" value="ATTiny84"/>
-<part name="SW1" library="PiB_switches" deviceset="SWITCH_SPDT" device="_RA_SMD_300MA-4V_6.7L-2.6W" value="300mA/4V"/>
+<part name="MCU1" library="PiB_ic_microcontrollers" deviceset="ATTINY84" device="_SOIC-14_NO_SILK" package3d_urn="urn:adsk.eagle:package:2967721/1" value="ATtiny84"/>
+<part name="SW1" library="PiB_switches" deviceset="SWITCH_SPDT" device="_RA_SMD_300MA-4V_6.7L-2.6W" package3d_urn="urn:adsk.eagle:package:2959400/2" value="300mA/4V"/>
 <part name="GND1" library="PiB_power_symbols" deviceset="GND" device=""/>
 <part name="GND3" library="PiB_power_symbols" deviceset="GND" device=""/>
-<part name="BATT1" library="PiB_batteries" deviceset="BATTERY_COIN-CELL" device="_SMD_3V_20MM" value="3V/225mAh"/>
-<part name="C1" library="PiB_capacitors" deviceset="10UF" device="_CER_SMD-0402_10V-20%" value="10uF/10V"/>
+<part name="BATT1" library="PiB_batteries" deviceset="BATTERY_COIN-CELL" device="_SMD_3V_20MM" package3d_urn="urn:adsk.eagle:package:2959529/4" value="225mAh/3V"/>
+<part name="C1" library="PiB_capacitors" deviceset="10UF" device="_CER_SMD-0402_6.3V-20%" package3d_urn="urn:adsk.eagle:package:2886515/1" value="10uF/6.3V"/>
 <part name="GND4" library="PiB_power_symbols" deviceset="GND" device=""/>
-<part name="C2" library="PiB_capacitors" deviceset="10UF" device="_CER_SMD-0402_10V-20%" value="10uF/10V"/>
+<part name="C2" library="PiB_capacitors" deviceset="10UF" device="_CER_SMD-0402_6.3V-20%" package3d_urn="urn:adsk.eagle:package:2886515/1" value="10uF/6.3V"/>
 <part name="GND5" library="PiB_power_symbols" deviceset="GND" device=""/>
 </parts>
@@
 <wire x1="-914.4" y1="-160.02" x2="-914.4" y2="-152.4" width="0.1524" layer="91"/>
 <pinref part="BATT1" gate="G$1" pin="+"/>
-<pinref part="SW1" gate="G$1" pin="2"/>
+<pinref part="SW1" gate="G$1" pin="P"/>
 <wire x1="-906.78" y1="-152.4" x2="-914.4" y2="-152.4" width="0.1524" layer="91"/>
 </segment>
@@
 <net name="N$11" class="0">
 <segment>
-<pinref part="SW1" gate="G$1" pin="3"/>
+<pinref part="SW1" gate="G$1" pin="S2"/>
 <pinref part="MCU1" gate="G$1" pin="VCC"/>
 <wire x1="-899.16" y1="-154.94" x2="-894.08" y2="-154.94" width="0.1524" layer="91"/>
@@
 </schematic>
 </drawing>
+<compatibility>
+<note version="8.3" severity="warning">
+Since Version 8.3, EAGLE supports URNs for individual library
+assets (packages, symbols, and devices). The URNs of those assets
+will not be understood (or retained) with this version.
+</note>
+<note version="8.3" severity="warning">
+Since Version 8.3, EAGLE supports the association of 3D packages
+with devices in libraries, schematics, and board files. Those 3D
+packages will not be understood (or retained) with this version.
+</note>
+</compatibility>
 </eagle>
